File: hw/pcb/pico_12vrgb_controller.kicad_pcb (KiCad board)
At the start: 2 copper layers, 101 x 31.8 mm, 20 parts, among them J1 Conn_01x04_RGB, J2 Conn_01x04_RGB, J3 Conn_01x04_RGB, J4 Conn_01x04_RGB, J5 Sata_15pin_Power, Q1 DMG2302U, Q10 DMG2302U, Q11 DMG2302U, Q12 DMG2302U, Q2 DMG2302U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

Commit message: Update SATA footprint based on physical part
Update minor dimensions in the 3D model, fix solder mask covering the
holes in the footprint, and add the repository URL to the board.
Other:
- board text added: "https://github.com/bluekeyes/pico-12vrgb-hid-controller"
Changed lines of the file:
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@@
+        (effects (font (size 1 1) (thickness 0.15)))
+    )
+    (fp_text user "B" (at 2.286 7.62 unlocked) (layer "F.SilkS")
+        (effects (font (size 1 1) (thickness 0.15)))
+    )
+    (fp_text user "G" (at 2.286 2.54 unlocked) (layer "F.SilkS")
         (effects (font (size 1 1) (thickness 0.15)))
     )
     (fp_text user "R" (at 2.286 5.08 unlocked) (layer "F.SilkS")
-        (effects (font (size 1 1) (thickness 0.15)))
-    )
-    (fp_text user "B" (at 2.286 7.62 unlocked) (layer "F.SilkS")
-        (effects (font (size 1 1) (thickness 0.15)))
-    )
-    (fp_text user "G" (at 2.286 2.54 unlocked) (layer "F.SilkS")
         (effects (font (size 1 1) (thickness 0.15)))
     )
@@
         (effects (font (size 1 1) (thickness 0.15)))
     )
+    (fp_text user "R" (at -2.413 5.08 unlocked) (layer "F.SilkS")
+        (effects (font (size 1 1) (thickness 0.15)))
+    )
     (fp_text user "B" (at -2.413 7.62 unlocked) (layer "F.SilkS")
         (effects (font (size 1 1) (thickness 0.15)))
     )
     (fp_text user "G" (at -2.413 2.54 unlocked) (layer "F.SilkS")
-        (effects (font (size 1 1) (thickness 0.15)))
-    )
-    (fp_text user "R" (at -2.413 5.08 unlocked) (layer "F.SilkS")
         (effects (font (size 1 1) (thickness 0.15)))
     )
@@
         (effects (font (size 1 1) (thickness 0.15)))
     )
+    (fp_text user "R" (at -2.413 5.08 unlocked) (layer "F.SilkS")
+        (effects (font (size 1 1) (thickness 0.15)))
+    )
+    (fp_text user "G" (at -2.413 2.54 unlocked) (layer "F.SilkS")
+        (effects (font (size 1 1) (thickness 0.15)))
+    )
     (fp_text user "B" (at -2.413 7.62 unlocked) (layer "F.SilkS")
-        (effects (font (size 1 1) (thickness 0.15)))
-    )
-    (fp_text user "R" (at -2.413 5.08 unlocked) (layer "F.SilkS")
-        (effects (font (size 1 1) (thickness 0.15)))
-    )
-    (fp_text user "G" (at -2.413 2.54 unlocked) (layer "F.SilkS")
         (effects (font (size 1 1) (thickness 0.15)))
     )
@@
     (fp_line (start 15.25 -3.67) (end 15.25 7.72)
       (stroke (width 0.12) (type solid)) (layer "F.SilkS"))
-    (pad "" np_thru_hole circle (at -13.4 7.22 90) (size 1.2 1.2) (drill 1.2) (layers "F&B.Cu"))
-    (pad "" np_thru_hole circle (at 13.4 7.22 90) (size 1.2 1.2) (drill 1.2) (layers "F&B.Cu"))
+    (pad "" np_thru_hole circle (at -13.4 7.22 90) (size 1.2 1.2) (drill 1.2) (layers "F&B.Cu" "*.Mask"))
+    (pad "" np_thru_hole circle (at 13.4 7.22 90) (size 1.2 1.2) (drill 1.2) (layers "F&B.Cu" "*.Mask"))
     (pad "1" thru_hole circle (at -8.5 0 90) (size 1 1) (drill 0.65) (layers "*.Cu" "*.Mask")
       (net 29 "unconnected-(J5-3V3-Pad1)") (pinfunction "3V3") (pintype "passive+no_connect"))
@@
         (effects (font (size 1 1) (thickness 0.15)))
     )
-    (fp_text user "Copper Keepouts shown on Dwgs layer" (at 0.1 -30.2 90) (layer "Cmts.User")
+    (fp_text user "Copper Keepouts shown on Dwgs layer" (at 0.1 -30.2 90) (layer "Cmts.User") hide
         (effects (font (size 1 1) (thickness 0.15)))
     )
@@
     )
   )
-  (gr_rect (start 123.4948 78.9178) (end 125.1458 73.66)
+  (gr_rect (start 123.4948 73.66) (end 125.1458 78.9178)
     (stroke (width 0.127) (type solid)) (fill none) (layer "F.SilkS"))
   (gr_rect (start 71.501 89.662) (end 75.819 91.313)
@@
   (gr_text "v1" (at 71.755 63.5) (layer "F.Cu")
     (effects (font (size 1.5 1.5) (thickness 0.3) bold) (justify left bottom))
+  )
+  (gr_text "https://github.com/bluekeyes/pico-12vrgb-hid-controller" (at 117.475 90.17) (layer "B.SilkS")
+    (effects (font (size 1 1) (thickness 0.15)) (justify left bottom mirror))
   )
   (gr_text "UART" (at 73.66 90.6272) (layer "F.SilkS")
@@
     (connect_pads yes (clearance 0.254))
     (min_thickness 0.254) (filled_areas_thickness no)
-    (fill yes (thermal_gap 0.508) (thermal_bridge_width 0.508))
+    (fill yes (thermal_gap 0.508) (thermal_bridge_width 0.6096))
     (polygon
       (pts
